Commit message: 2024/9/18 update

File: kataude_description/urdf/kataude.xacro (robot description, xacro)
@@ -1,11 +1,12 @@
 <?xml version="1.0" ?>
 <robot name="kataude" xmlns:xacro="http://www.ros.org/wiki/xacro">
-<xacro:include filename="$(find kataude_description)/urdf/materials.xacro" />
-<xacro:include filename="$(find kataude_description)/urdf/kataude.trans" />
-<xacro:include filename="$(find kataude_description)/urdf/kataude.gazebo" />
+<!-- <link name="dummy">
+   </link> -->
+<link name="world" />
 <link name="base_link">
   <inertial>
     <origin xyz="-0.15278443948564172 -1.646071389736825e-05 1.9943676527636152" rpy="0 0 0"/>
-    <mass value="3.145965262261491"/>
+    <!-- <mass value="3.145965262261491"/> -->
+    <mass value="1000000"/>
     <inertia ixx="0.001806" iyy="0.005212" izz="0.004982" ixy="-0.0" iyz="0.0" ixz="4e-06"/>
   </inertial>
@@ -27,5 +28,6 @@
   <inertial>
     <origin xyz="2.3936065328189482e-05 0.06873152009023258 -0.3984141268400523" rpy="0 0 0"/>
-    <mass value="142.51149550389982"/>
+    <!-- <mass value="142.51149550389982"/> -->
+    <mass value="1.4251149550389982"/>
     <inertia ixx="5.64702" iyy="5.488361" izz="0.635098" ixy="-0.0" iyz="-0.000188" ixz="2.8e-05"/>
   </inertial>
@@ -47,5 +49,6 @@
   <inertial>
     <origin xyz="0.024533563447407203 -0.00021381174077944674 -0.0631193250864" rpy="0 0 0"/>
-    <mass value="0.09824516357620273"/>
+    <!-- <mass value="0.09824516357620273"/> -->
+    <mass value="0.164"/>
     <inertia ixx="6.2e-05" iyy="5.8e-05" izz="2.8e-05" ixy="-0.0" iyz="-0.0" ixz="-2e-06"/>
   </inertial>
@@ -67,5 +70,6 @@
   <inertial>
     <origin xyz="-9.00741698207086e-05 -0.02460604325871079 -0.04241777280246267" rpy="0 0 0"/>
-    <mass value="0.5291067052461904"/>
+    <!-- <mass value="0.5291067052461904"/> -->
+    <mass value="0.164"/>
     <inertia ixx="0.000219" iyy="0.00018" izz="0.000224" ixy="-1e-06" iyz="-6e-06" ixz="-0.0"/>
   </inertial>
@@ -87,5 +91,6 @@
   <inertial>
     <origin xyz="-0.001267246990176496 0.00020718172021483958 0.029980098166622282" rpy="0 0 0"/>
-    <mass value="4.659806299364297"/>
+    <!-- <mass value="4.659806299364297"/> -->
+    <mass value="1.659806299364297"/>
     <inertia ixx="0.006381" iyy="0.074421" izz="0.076997" ixy="7.7e-05" iyz="1.2e-05" ixz="-0.006229"/>
   </inertial>
@@ -107,5 +112,6 @@
   <inertial>
     <origin xyz="0.00010929466551301559 0.06821266521028407 -0.3727168964631816" rpy="0 0 0"/>
-    <mass value="131.66138695773583"/>
+    <!-- <mass value="131.66138695773583"/> -->
+    <mass value="1.3166138695773583"/>
     <inertia ixx="4.458919" iyy="4.313539" izz="0.590679" ixy="0.0" iyz="-0.00075" ixz="-0.000184"/>
   </inertial>
@@ -127,5 +133,6 @@
   <inertial>
     <origin xyz="-0.0002450048864300891 2.0149603131389355e-05 -0.03209129443533182" rpy="0 0 0"/>
-    <mass value="0.09211846580456283"/>
+    <!-- <mass value="0.09211846580456283"/> -->
+    <mass value="0.170"/>
     <inertia ixx="3.9e-05" iyy="4.6e-05" izz="2.4e-05" ixy="0.0" iyz="-0.0" ixz="-0.0"/>
   </inertial>
@@ -147,5 +154,5 @@
   <inertial>
     <origin xyz="-0.019092930378784956 -0.008786732838234303 -0.03526207180079688" rpy="0 0 0"/>
-    <mass value="0.3618135799855471"/>
+    <mass value="0.27970437781382335"/>
     <inertia ixx="0.0003" iyy="0.000362" izz="0.000133" ixy="0.0" iyz="2.3e-05" ixz="1e-06"/>
   </inertial>
@@ -184,4 +191,20 @@
   </collision>
 </link>
+<!-- <joint name="dummy_joint" type="fixed">
+     <parent link="dummy"/>
+     <child link="base_link"/>
+   </joint> -->
+<joint name="world_joint" type="fixed">
+    <parent link="world"/>
+    <child link="base_link"/>
+    <origin xyz="0 0 0" rpy="0 0 0"/>
+  </joint>
+<joint name="ShoulderJoint1" type="revolute">
+  <origin xyz="-0.2215 -2e-05 1.99849" rpy="0 0 0"/>
+  <parent link="base_link"/>
+  <child link="Shoulder_Servo3_1"/>
+  <axis xyz="1.0 -0.0 -0.0"/>
+  <limit upper="3.14" lower="-3.14" effort="100" velocity="100"/>
+</joint>
 <joint name="ShoulderJoint2" type="revolute">
   <origin xyz="-0.081 -0.06897 0.01803" rpy="0 0 0"/>
@@ -189,5 +212,30 @@
   <child link="UpperArm_1"/>
   <axis xyz="0.0 1.0 0.0"/>
-  <limit upper="3.141593" lower="0.0" effort="100" velocity="100"/>
+  <limit upper="3.141593" lower ="0.0" effort="100" velocity="100"/>
+</joint>
+<!--
+<transmission name="ShoulderJoint2_trans">
+    <type>transmission_interface/SimpleTransmission</type>
+    <joint name="ShoulderJoint2">
+      <hardwareInterface>hardware_interface/EffortJointInterface</hardwareInterface>
+    </joint>
+    <actuator name="ShoulderJoint2_motor">
+       <hardwareInterface>hardware_interface/EffortJointInterface</hardwareInterface>
+       <mechanismReduction>1</mechanismReduction>
+    </actuator>
+</transmission>
+-->
+<joint name="ElbowJoint" type="revolute">
+  <origin xyz="3.4e-05 -9.2e-05 -0.765979" rpy="0 0 0"/>
+  <parent link="UpperArm_1"/>
+  <child link="ForeArm_1"/>
+  <axis xyz="-0.0 1.0 0.0"/>
+  <limit upper="1.570796" lower="-1.570796" effort="100" velocity="100"/>
+</joint>
+<joint name="xm540_1" type="continuous">
+  <origin xyz="0.00514 0.068198 -0.743224" rpy="0 0 0"/>
+  <parent link="ForeArm_1"/>
+  <child link="XM540_270R_2_1"/>
+  <axis xyz="0.0 -0.0 -1.0"/>
 </joint>
 <joint name="xm540_2" type="revolute">
@@ -205,24 +253,4 @@
   <limit upper="1.570796" lower="-1.570796" effort="100" velocity="100"/>
 </joint>
-<joint name="ShoulderJoint1" type="revolute">
-  <origin xyz="-0.2215 -2e-05 1.99849" rpy="0 0 0"/>
-  <parent link="base_link"/>
-  <child link="Shoulder_Servo3_1"/>
-  <axis xyz="1.0 -0.0 -0.0"/>
-  <limit upper="1.570796" lower="-1.570796" effort="100" velocity="100"/>
-</joint>
-<joint name="ElbowJoint" type="revolute">
-  <origin xyz="3.4e-05 -9.2e-05 -0.765979" rpy="0 0 0"/>
-  <parent link="UpperArm_1"/>
-  <child link="ForeArm_1"/>
-  <axis xyz="-0.0 1.0 0.0"/>
-  <limit upper="1.570796" lower="-1.570796" effort="100" velocity="100"/>
-</joint>
-<joint name="xm540_1" type="continuous">
-  <origin xyz="0.00514 0.068198 -0.743224" rpy="0 0 0"/>
-  <parent link="ForeArm_1"/>
-  <child link="XM540_270R_2_1"/>
-  <axis xyz="0.0 -0.0 -1.0"/>
-</joint>
 <joint name="EndEffecter1" type="revolute">
   <origin xyz="0.016974 -0.043809 -0.046242" rpy="0 0 0"/>
@@ -232,5 +260,5 @@
   <limit upper="0.0" lower="-1.047198" effort="100" velocity="100"/>
 </joint>
-<joint name="Endeffecter2" type="revolute">
+<joint name="EndEffecter2" type="revolute">
   <origin xyz="0.016974 -0.011809 -0.046242" rpy="0 0 0"/>
   <parent link="mikata_arm_1"/>
@@ -239,3 +267,6 @@
   <limit upper="1.047198" lower="0.0" effort="100" velocity="100"/>
 </joint>
+<xacro:include filename="$(find kataude_description)/urdf/materials.xacro" />
+<xacro:include filename="$(find kataude_description)/urdf/kataude.trans" />
+<xacro:include filename="$(find kataude_description)/urdf/kataude.gazebo" />
 </robot>
