Commit message: update

File: souwan_description/urdf/souwan.xacro (robot description, xacro)
@@ -26,4 +26,33 @@
   </collision>
 </link>
+<!-- 円柱リンク -->
+<link name="cylinder_link">
+  <inertial>
+    <origin xyz="0 0 1.5" rpy="0 0 0"/>
+    <mass value="1.0"/>
+    <inertia ixx="0.1" iyy="0.1" izz="0.2" ixy="0" ixz="0" iyz="0"/>
+  </inertial>
+  <visual>
+    <origin xyz="0 0 1.0" rpy="0 0 0"/>
+    <geometry>
+      <cylinder radius="0.2" length="2.0"/>
+    </geometry>
+    <material>
+      <color rgba="0.8 0.2 0.2 1.0"/>
+    </material>
+  </visual>
+  <collision>
+    <origin xyz="0 0 1.0" rpy="0 0 0"/>
+    <geometry>
+      <cylinder radius="0.2" length="2.0"/>
+    </geometry>
+  </collision>
+</link>
+<!-- base_link に固定された円柱ジョイント -->
+<joint name="cylinder_joint" type="fixed">
+  <parent link="base_link"/>
+  <child link="cylinder_link"/>
+  <origin xyz="0 0 1.0" rpy="0 0 0"/>
+</joint>
 <link name="UpperArm_1">
   <inertial>
@@ -557,5 +586,5 @@
   <axis xyz="-0.0 0.0 -1.0"/>
 </joint>
-<joint name="Endeffector2" type="revolute">
+<joint name="EndEffector2" type="revolute">
   <origin xyz="-0.016974 0.043809 -0.046242" rpy="0 0 0"/>
   <parent link="mikata_arm_1"/>
@@ -564,5 +593,5 @@
   <limit upper="0.0" lower="-1.047198" effort="100" velocity="100"/>
 </joint>
-<joint name="Endeffector1" type="revolute">
+<joint name="EndEffector1" type="revolute">
   <origin xyz="-0.016974 0.011809 -0.046242" rpy="0 0 0"/>
   <parent link="mikata_arm_1"/>
@@ -571,4 +600,9 @@
   <limit upper="1.047198" lower="0.0" effort="100" velocity="100"/>
 </joint>
+<joint name="tactile1" type="fixed">
+  <origin xyz="-0.075048 -0.068708 -0.391937" rpy="0 0 0"/>
+  <parent link="UpperArm_1"/>
+  <child link="tactile1_1"/>
+</joint>
 <joint name="tactile2" type="fixed">
   <origin xyz="-0.075048 -0.018708 -0.672937" rpy="0 0 0"/>
@@ -576,8 +610,8 @@
   <child link="tactile2_1"/>
 </joint>
-<joint name="tactile1" type="fixed">
-  <origin xyz="-0.075048 -0.068708 -0.391937" rpy="0 0 0"/>
-  <parent link="UpperArm_1"/>
-  <child link="tactile1_1"/>
+<joint name="tactile3" type="fixed">
+  <origin xyz="-0.075141 -0.018197 -0.110984" rpy="0 0 0"/>
+  <parent link="ForeArm_1"/>
+  <child link="tactile3_1"/>
 </joint>
 <joint name="tactile4" type="fixed">
@@ -585,9 +619,4 @@
   <parent link="ForeArm_1"/>
   <child link="tactile4_1"/>
-</joint>
-<joint name="tactile3" type="fixed">
-  <origin xyz="-0.075141 -0.018197 -0.110984" rpy="0 0 0"/>
-  <parent link="ForeArm_1"/>
-  <child link="tactile3_1"/>
 </joint>
 <joint name="ShoulderJoint2R" type="revolute">
@@ -645,5 +674,5 @@
   <child link="tactile4R_1"/>
 </joint>
-<joint name="Endeffetor1R" type="revolute">
+<joint name="EndEffector1R" type="revolute">
   <origin xyz="-0.020926 -0.039191 -0.046242" rpy="0 0 0"/>
   <parent link="mikata_armR_1"/>
@@ -652,5 +681,5 @@
   <limit upper="1.047198" lower="0.0" effort="100" velocity="100"/>
 </joint>
-<joint name="Endeffecter2R" type="revolute">
+<joint name="EndEffector2R" type="revolute">
   <origin xyz="-0.017026 -0.007191 -0.046242" rpy="0 0 0"/>
   <parent link="mikata_armR_1"/>
